File: kicad/touch-zigbee/touch-zigbee.kicad_sch (KiCad schematic)
At the start: 19 parts, among them Q1 2N7000, Q2 2N7000, Q3 TP0610L, U1 7333-A-TO92, U3 ATtiny84A-PU

Commit message: update kicad schematic
Parts:
- Capacitive_Sensor_CJMCU-1010: symbol Connector:Conn_01x03_Female -> touch-zigbee-rescue:Conn_01x03_Female-Connector
- Power1: symbol Connector:Conn_01x02_Female -> touch-zigbee-rescue:Conn_01x02_Female-Connector
